File: kicad/io.kicad_sch (KiCad schematic)
At the start: 11 parts, among them J2 UART, P1 Mini-DIN_6pins_ver3, U13 uSD adapter, U14 8259, U16 16550, U17 T6963C

Commit message: New PCB (add MCB line)
Parts:
- added R2: 10K, Resistor_THT:R_Axial_DIN0204_L3.6mm_D1.6mm_P7.62mm_Horizontal, symbol Device:R
Connections:
- net GND: now also R2.1
- net MCB: now reaches U?.4 (PA0)
- net MCB: now also R2.2
- no-connect marks 43 -> 42
Changed lines of the file:
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@@
   (junction (at 332.74 102.87) (diameter 0) (color 0 0 0 0)
+  )
+  (junction (at 246.38 48.26) (diameter 0) (color 0 0 0 0)
   )
   (junction (at 177.8 160.02) (diameter 0) (color 0 0 0 0)
@@
   (no_connect (at 248.92 96.52))
   (no_connect (at 241.3 50.8))
-  (no_connect (at 241.3 48.26))
   (no_connect (at 347.98 41.91))
   (no_connect (at 347.98 54.61))
@@
     (stroke (width 0) (type default))
   )
+  (wire (pts (xy 246.38 48.26) (xy 251.46 48.26))
+    (stroke (width 0) (type default))
+  )
   (wire (pts (xy 83.82 138.43) (xy 96.52 138.43))
     (stroke (width 0) (type default))
@@
   )
   (bus (pts (xy 320.04 44.45) (xy 320.04 41.91))
+    (stroke (width 0) (type default))
+  )
+  (wire (pts (xy 241.3 48.26) (xy 246.38 48.26))
     (stroke (width 0) (type default))
   )
@@
     (property "Intersheetrefs" "${INTERSHEET_REFS}" (at 191.7578 71.12 0)
       (effects (font (size 1.27 1.27)) (justify right) hide)
+    )
+  )
+  (global_label "MCB" (shape output) (at 251.46 48.26 0) (fields_autoplaced)
+    (effects (font (size 1.27 1.27)) (justify left))
+    (property "Intersheetrefs" "${INTERSHEET_REFS}" (at 258.4366 48.26 0)
+      (effects (font (size 1.27 1.27)) (justify left) hide)
     )
   )
@@
     )
   )
+  (symbol (lib_id "power:GND") (at 246.38 55.88 0) (unit 1)
+    (in_bom yes) (on_board yes) (dnp no) (fields_autoplaced)
+    (property "Reference" "#PWR?" (at 246.38 62.23 0)
+      (effects (font (size 1.27 1.27)) hide)
+    )
+    (property "Value" "GND" (at 246.38 60.96 0)
+      (effects (font (size 1.27 1.27)))
+    )
+    (property "Footprint" "" (at 246.38 55.88 0)
+      (effects (font (size 1.27 1.27)) hide)
+    )
+    (property "Datasheet" "" (at 246.38 55.88 0)
+      (effects (font (size 1.27 1.27)) hide)
+    )
+    (pin "1")
+    (instances
+      (project "main"
+        (path "/590a4a95-7c0e-40dd-8637-8ee29cb6972a"
+          (reference "#PWR?") (unit 1)
+        )
+        (path "/590a4a95-7c0e-40dd-8637-8ee29cb6972a/3a7ee20c-9aab-4bcf-8400-2397304f0b30"
+          (reference "#PWR026") (unit 1)
+        )
+      )
+    )
+  )
   (symbol (lib_id "power:+5V") (at 337.82 29.21 0) (unit 1)
     (in_bom yes) (on_board yes) (dnp no) (fields_autoplaced)
@@
         )
       )
+    )
+  )
+  (symbol (lib_id "Device:R") (at 246.38 52.07 180) (unit 1)
+    (in_bom yes) (on_board yes) (dnp no) (fields_autoplaced)
+    (property "Reference" "R2" (at 248.92 50.8 0)
+      (effects (font (size 1.27 1.27)) (justify right))
+    )
+    (property "Value" "10K" (at 248.92 53.34 0)
+      (effects (font (size 1.27 1.27)) (justify right))
+    )
+    (property "Footprint" "Resistor_THT:R_Axial_DIN0204_L3.6mm_D1.6mm_P7.62mm_Horizontal" (at 248.158 52.07 90)
+      (effects (font (size 1.27 1.27)) hide)
+    )
+    (property "Datasheet" "~" (at 246.38 52.07 0)
+      (effects (font (size 1.27 1.27)) hide)
+    )
+    (pin "1")
+    (pin "2")
+    (instances
+      (project "main"
+        (path "/590a4a95-7c0e-40dd-8637-8ee29cb6972a"
+          (reference "R2") (unit 1)
+        )
+        (path "/590a4a95-7c0e-40dd-8637-8ee29cb6972a/3a7ee20c-9aab-4bcf-8400-2397304f0b30"
+          (reference "R1") (unit 1)
+        )
+      )
